File: src/eagle/pub.sch (EAGLE design)
At the start: 26 parts, among them IC1 PIC18F25K50, SW1 EC12E_SW

Commit message: Tweaked PCB slightly
Parts:
- JP1: value PICKIT -> MIKROPROG; device pinhead:PINHD-1X6 -> pub:PINHD-1X5/90
- JP2: value MIKROPROG -> PICKKIT; device SparkFun-Connectors:M05PTH -> pub:PINHD-1X6/90
Connections:
- net GND: now also JP1.5, JP2.3, JP3.MNT1, JP3.MNT2, JP3.MNT3, JP3.MNT4; no longer JP1.3, JP2.5
- net N$10: now also JP1.4, JP2.1; no longer JP1.1, JP2.4
- net N$7: now also JP1.1, JP2.2; no longer JP1.2, JP2.1
- net N$8: now also JP1.2, JP2.5; no longer JP1.5, JP2.2
- net N$9: now also JP1.3, JP2.4; no longer JP1.4, JP2.3
Other:
- moved on the sheet: C1

Commit message: Fixed PCB to match code. Rotary button on RB6
Parts:
- added RB3: TPB1,27, testpad:TPB1,27
Connections:
- removed net RA1: IC1.AN9/RB3, SW1G$2.2
- net GND: now also IC1.AN9/RB3, RB3.TP
- net N$8: now also SW1G$2.2
Other:
- moved on the sheet: SW1
Changed lines of the file:
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@@
 <?xml version="1.0" encoding="utf-8"?>
 <!DOCTYPE eagle SYSTEM "eagle.dtd">
-<eagle version="6.5.0">
+<eagle version="6.6.0">
 <drawing>
 <settings>
@@
 <grid distance="0.1" unitdist="inch" unit="inch" style="lines" multiple="1" display="yes" altdistance="0.01" altunitdist="inch" altunit="inch"/>
 <layers>
-<layer number="1" name="Top" color="11" fill="1" visible="yes" active="no"/>
-<layer number="2" name="Route2" color="1" fill="3" visible="yes" active="no"/>
-<layer number="3" name="Route3" color="4" fill="3" visible="yes" active="no"/>
-<layer number="14" name="Route14" color="1" fill="6" visible="yes" active="no"/>
-<layer number="15" name="Route15" color="4" fill="6" visible="yes" active="no"/>
-<layer number="16" name="Bottom" color="9" fill="1" visible="yes" active="no"/>
-<layer number="17" name="Pads" color="2" fill="1" visible="yes" active="no"/>
-<layer number="18" name="Vias" color="12" fill="1" visible="yes" active="no"/>
-<layer number="19" name="Unrouted" color="6" fill="1" visible="yes" active="no"/>
-<layer number="20" name="Dimension" color="15" fill="1" visible="yes" active="no"/>
-<layer number="21" name="tPlace" color="15" fill="1" visible="yes" active="no"/>
-<layer number="22" name="bPlace" color="23" fill="1" visible="yes" active="no"/>
-<layer number="23" name="tOrigins" color="15" fill="1" visible="yes" active="no"/>
-<layer number="24" name="bOrigins" color="23" fill="1" visible="yes" active="no"/>
-<layer number="25" name="tNames" color="15" fill="1" visible="yes" active="no"/>
-<layer number="26" name="bNames" color="23" fill="1" visible="yes" active="no"/>
-<layer number="27" name="tValues" color="15" fill="1" visible="yes" active="no"/>
-<layer number="28" name="bValues" color="23" fill="1" visible="yes" active="no"/>
+<layer number="1" name="Top" color="11" fill="1" visible="no" active="no"/>
+<layer number="2" name="Route2" color="1" fill="3" visible="no" active="no"/>
+<layer number="3" name="Route3" color="4" fill="3" visible="no" active="no"/>
+<layer number="14" name="Route14" color="1" fill="6" visible="no" active="no"/>
+<layer number="15" name="Route15" color="4" fill="6" visible="no" active="no"/>
+<layer number="16" name="Bottom" color="9" fill="1" visible="no" active="no"/>
+<layer number="17" name="Pads" color="2" fill="1" visible="no" active="no"/>
+<layer number="18" name="Vias" color="12" fill="1" visible="no" active="no"/>
+<layer number="19" name="Unrouted" color="6" fill="1" visible="no" active="no"/>
+<layer number="20" name="Dimension" color="15" fill="1" visible="no" active="no"/>
+<layer number="21" name="tPlace" color="15" fill="1" visible="no" active="no"/>
+<layer number="22" name="bPlace" color="23" fill="1" visible="no" active="no"/>
+<layer number="23" name="tOrigins" color="15" fill="1" visible="no" active="no"/>
+<layer number="24" name="bOrigins" color="23" fill="1" visible="no" active="no"/>
+<layer number="25" name="tNames" color="15" fill="1" visible="no" active="no"/>
+<layer number="26" name="bNames" color="23" fill="1" visible="no" active="no"/>
+<layer number="27" name="tValues" color="15" fill="1" visible="no" active="no"/>
+<layer number="28" name="bValues" color="23" fill="1" visible="no" active="no"/>
 <layer number="29" name="tStop" color="7" fill="3" visible="no" active="no"/>
 <layer number="30" name="bStop" color="7" fill="6" visible="no" active="no"/>
@@
 <layer number="35" name="tGlue" color="7" fill="4" visible="no" active="no"/>
 <layer number="36" name="bGlue" color="7" fill="5" visible="no" active="no"/>
-<layer number="37" name="tTest" color="7" fill="1" visible="yes" active="no"/>
-<layer number="38" name="bTest" color="7" fill="1" visible="yes" active="no"/>
+<layer number="37" name="tTest" color="7" fill="1" visible="no" active="no"/>
+<layer number="38" name="bTest" color="7" fill="1" visible="no" active="no"/>
 <layer number="39" name="tKeepout" color="3" fill="11" visible="no" active="no"/>
 <layer number="40" name="bKeepout" color="1" fill="11" visible="no" active="no"/>
@@
 <layer number="44" name="Drills" color="7" fill="1" visible="no" active="no"/>
 <layer number="45" name="Holes" color="7" fill="1" visible="no" active="no"/>
-<layer number="46" name="Milling" color="3" fill="1" visible="yes" active="no"/>
-<layer number="47" name="Measures" color="7" fill="1" visible="yes" active="no"/>
-<layer number="48" name="Document" color="7" fill="1" visible="yes" active="no"/>
-<layer number="49" name="Reference" color="7" fill="1" visible="yes" active="no"/>
-<layer number="50" name="dxf" color="7" fill="1" visible="yes" active="no"/>
-<layer number="51" name="tDocu" color="7" fill="1" visible="yes" active="no"/>
-<layer number="52" name="bDocu" color="7" fill="1" visible="yes" active="no"/>
-<layer number="53" name="tGND_GNDA" color="7" fill="9" visible="yes" active="no"/>
-<layer number="54" name="bGND_GNDA" color="1" fill="9" visible="yes" active="no"/>
-<layer number="56" name="wert" color="7" fill="1" visible="yes" active="no"/>
-<layer number="57" name="tCAD" color="7" fill="1" visible="yes" active="no"/>
+<layer number="46" name="Milling" color="3" fill="1" visible="no" active="no"/>
+<layer number="47" name="Measures" color="7" fill="1" visible="no" active="no"/>
+<layer number="48" name="Document" color="7" fill="1" visible="no" active="no"/>
+<layer number="49" name="Reference" color="7" fill="1" visible="no" active="no"/>
+<layer number="50" name="dxf" color="7" fill="1" visible="no" active="no"/>
+<layer number="51" name="tDocu" color="7" fill="1" visible="no" active="no"/>
+<layer number="52" name="bDocu" color="7" fill="1" visible="no" active="no"/>
+<layer number="53" name="tGND_GNDA" color="7" fill="9" visible="no" active="no"/>
+<layer number="54" name="bGND_GNDA" color="1" fill="9" visible="no" active="no"/>
+<layer number="56" name="wert" color="7" fill="1" visible="no" active="no"/>
+<layer number="57" name="tCAD" color="7" fill="1" visible="no" active="no"/>
 <layer number="91" name="Nets" color="2" fill="1" visible="yes" active="yes"/>
 <layer number="92" name="Busses" color="1" fill="1" visible="yes" active="yes"/>
@@
 <part name="JP1" library="pub" deviceset="PINHD-1X5" device="/90" value="MIKROPROG"/>
 <part name="JP2" library="pub" deviceset="PINHD-1X6" device="/90" value="PICKKIT"/>
+<part name="RB3" library="testpad" deviceset="TP" device="B1,27"/>
 </parts>
 <sheets>
@@
 <instance part="IC1" gate="G$1" x="2.54" y="40.64"/>
 <instance part="SW1" gate="G$1" x="66.04" y="50.8" rot="R90"/>
-<instance part="SW1" gate="G$2" x="63.5" y="43.18"/>
+<instance part="SW1" gate="G$2" x="63.5" y="58.42" smashed="yes">
+<attribute name="PART" x="58.42" y="63.5" size="1.27" layer="95"/>
+<attribute name="VALUE" x="71.12" y="58.42" size="1.27" layer="96"/>
+</instance>
 <instance part="GND1" gate="1" x="78.74" y="-2.54"/>
 <instance part="GND2" gate="1" x="78.74" y="45.72"/>
@@
 <attribute name="VALUE" x="-5.842" y="91.44" size="1.778" layer="96"/>
 </instance>
+<instance part="RB3" gate="G$1" x="27.94" y="48.26" smashed="yes" rot="R270">
+<attribute name="NAME" x="29.21" y="46.99" size="1.778" layer="95"/>
+<attribute name="TP_SIGNAL_NAME" x="26.67" y="46.99" size="1.778" layer="97" rot="R270"/>
+</instance>
 </instances>
 <busses>
@@
 </segment>
 <segment>
-<pinref part="SW1" gate="G$2" pin="1"/>
 <pinref part="GND2" gate="1" pin="GND"/>
 <wire x1="78.74" y1="50.8" x2="78.74" y2="48.26" width="0.1524" layer="91"/>
@@
 <wire x1="68.58" y1="50.8" x2="78.74" y2="50.8" width="0.1524" layer="91"/>
 <junction x="68.58" y="50.8"/>
-<wire x1="68.58" y1="50.8" x2="68.58" y2="43.18" width="0.1524" layer="91"/>
 <wire x1="50.8" y1="86.36" x2="50.8" y2="66.04" width="0.1524" layer="91"/>
 <wire x1="50.8" y1="66.04" x2="68.58" y2="66.04" width="0.1524" layer="91"/>
-<wire x1="68.58" y1="66.04" x2="68.58" y2="50.8" width="0.1524" layer="91"/>
+<wire x1="68.58" y1="66.04" x2="68.58" y2="58.42" width="0.1524" layer="91"/>
 <pinref part="JP1" gate="A" pin="5"/>
 <pinref part="JP3" gate="G$1" pin="MNT1"/>
+<wire x1="68.58" y1="58.42" x2="68.58" y2="50.8" width="0.1524" layer="91"/>
 <wire x1="86.36" y1="30.48" x2="86.36" y2="50.8" width="0.1524" layer="91"/>
 <wire x1="86.36" y1="50.8" x2="78.74" y2="50.8" width="0.1524" layer="91"/>
@@
 <wire x1="-2.54" y1="66.04" x2="50.8" y2="66.04" width="0.1524" layer="91"/>
 <junction x="50.8" y="66.04"/>
+<pinref part="SW1" gate="G$2" pin="1"/>
+<junction x="68.58" y="58.42"/>
 </segment>
 <segment>
@@
 <wire x1="25.4" y1="43.18" x2="25.4" y2="45.72" width="0.1524" layer="91"/>
 <junction x="25.4" y="45.72"/>
+<pinref part="IC1" gate="G$1" pin="AN9/RB3"/>
+<pinref part="RB3" gate="G$1" pin="TP"/>
+<wire x1="20.32" y1="48.26" x2="25.4" y2="48.26" width="0.1524" layer="91"/>
+<wire x1="25.4" y1="45.72" x2="25.4" y2="48.26" width="0.1524" layer="91"/>
+<junction x="25.4" y="48.26"/>
 </segment>
 <segment>
@@
 <wire x1="20.32" y1="50.8" x2="58.42" y2="50.8" width="0.1524" layer="91"/>
 <wire x1="58.42" y1="50.8" x2="58.42" y2="48.26" width="0.1524" layer="91"/>
-</segment>
-</net>
-<net name="RA1" class="0">
-<segment>
-<pinref part="IC1" gate="G$1" pin="AN9/RB3"/>
-<wire x1="20.32" y1="48.26" x2="55.88" y2="48.26" width="0.1524" layer="91"/>
-<wire x1="55.88" y1="48.26" x2="55.88" y2="43.18" width="0.1524" layer="91"/>
-<pinref part="SW1" gate="G$2" pin="2"/>
-<wire x1="55.88" y1="43.18" x2="58.42" y2="43.18" width="0.1524" layer="91"/>
 </segment>
 </net>
@@
 <pinref part="JP2" gate="A" pin="5"/>
 <pinref part="JP1" gate="A" pin="2"/>
-</segment>
-</net>
+<pinref part="SW1" gate="G$2" pin="2"/>
+<wire x1="58.42" y1="58.42" x2="58.42" y2="55.88" width="0.1524" layer="91"/>
+<wire x1="58.42" y1="55.88" x2="43.18" y2="55.88" width="0.1524" layer="91"/>
+<junction x="43.18" y="55.88"/>
+</segment>
+</net>
