File: src/eagle/pub.sch (EAGLE design)
At the start: 27 parts, among them IC1 PIC18F25K50, SW1 EC12E_SW

Commit message: Fixed typo in PICKIT header.
How did I not see it spelled as PICKKIT? Sheesh!
Parts:
- JP2: value PICKKIT -> PICKIT
Changed lines of the file:
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@@
 <part name="JP3" library="pub" deviceset="USB-MINIB" device="-5PIN"/>
 <part name="JP1" library="pub" deviceset="PINHD-1X5" device="/90" value="MIKROPROG"/>
-<part name="JP2" library="pub" deviceset="PINHD-1X6" device="/90" value="PICKKIT"/>
+<part name="JP2" library="pub" deviceset="PINHD-1X6" device="/90" value="PICKIT"/>
 <part name="RB3" library="testpad" deviceset="TP" device="B1,27"/>
 </parts>
